File: Hardware/Shield 1.2/bombclock_1.3.brd (EAGLE design)
At the start: 68.6 x 53.3 mm, 42 parts, among them U1 ARDUINOR3-DIMENSION

Commit message: Updates
Updates
Parts:
- HT16K33: value (none) -> HT16K33
Changed lines of the file:
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@@
 <element name="R28" library="resistor" package="R0603" value="47K" x="53.34" y="29.21" rot="MR0"/>
 <element name="R29" library="resistor" package="R0603" value="47K" x="53.34" y="26.67" rot="MR0"/>
-<element name="HT16K33" library="microbuilder" package="SOP28_300MIL" value="" x="17.78" y="24.13" rot="MR270"/>
+<element name="HT16K33" library="microbuilder" package="SOP28_300MIL" value="HT16K33" x="17.78" y="24.13" rot="MR270"/>
 <element name="A2" library="microbuilder" package="SOLDERJUMPER_REFLOW_NOPASTE" value="" x="49.53" y="31.75" rot="MR0"/>
 <element name="R30" library="resistor" package="R0603" value="47K" x="53.34" y="31.75" rot="MR0"/>
