File: Hardware/Shield 1.2/bombclock_1.3.sch (EAGLE design)
At the start: 42 parts, among them U1 ARDUINOR3-DIMENSION

Commit message: Updates
Updates
Parts:
- HT16K33: value (none) -> HT16K33
Changed lines of the file:
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@@
 <part name="R28" library="resistor" deviceset="R-EU_" device="R0603" value="47K"/>
 <part name="R29" library="resistor" deviceset="R-EU_" device="R0603" value="47K"/>
-<part name="HT16K33" library="microbuilder" deviceset="HT16K33_SOP28" device=""/>
+<part name="HT16K33" library="microbuilder" deviceset="HT16K33_SOP28" device="" value="HT16K33"/>
 <part name="GND1" library="supply1" deviceset="GND" device=""/>
 <part name="A2" library="microbuilder" deviceset="SOLDERJUMPER" device="REFLOW_NOPASTE"/>
